File: MagneticSwitch_and_POT_Module/MagneticSwitch_and_POT_Module.kicad_pcb (KiCad board)
At the start: 4 copper layers, 114.3 x 85 mm, 87 parts, among them J1 Conn_01x06, J2 Conn_01x06, J3 Conn_01x06, U1 DRV5056A3QDBZR, U10 DRV5056A3QDBZR, U11 DRV5056A3QDBZR, U2 DRV5056A3QDBZR, U3 DRV5056A3QDBZR, U4 DRV5056A3QDBZR, U5 DRV5056A3QDBZR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

Commit message: Add comment.
Other:
- board text added: "UNIT: mm t:1.2(recommend)"
- board text removed: "t:1.2mm (recommend)"
Changed lines of the file:
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@@
 		)
 	)
-	(gr_text "t:1.2mm (recommend)"
-		(at 68.63 156.99 0)
+	(gr_text "UNIT: mm\nt:1.2(recommend)"
+		(at 183.74 71.41 0)
 		(layer "Cmts.User")
 		(effects
